File: HARDWARE/NeuroBytes_Tonic_Neuron.kicad_pcb (KiCad board)
At the start: 2 copper layers, 51.9 x 18 mm, 28 parts, among them P1 CONN_01X04, P2 CONN_01X04, P3 CONN_01X04, P4 JST_GH_5-pos, Q1 Q_NPN_BEC, Q2 Q_NPN_BEC, Q3 Q_NPN_BEC, SW1 SW_PUSH, U1 STM32L011Gx, U2 LD3985G33R

Commit message: finished routing with discrete NPN transitors and resistors
Routing:
- net Net-(Q2-Pad1): track 8.73 -> 24.9 mm, vias 1 -> 2
- net Net-(Q1-Pad1): track 14.9 -> 27.3 mm, vias 1 -> 2
- net LED_B: track 18.4 -> 26.5 mm, vias 1 -> 2
- net LED_R: track 0.02 -> 2.31 mm
- net LED_G: track 0.00 -> 2.18 mm
Changed lines of the file:
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@@
   (general
     (links 73)
-    (no_connects 16)
-    (area 153.199999 60.917456 205.198036 79.062409)
+    (no_connects 13)
+    (area 151.126667 58.081428 208.589752 82.489752)
     (thickness 1.6)
     (drawings 45)
-    (tracks 360)
+    (tracks 391)
     (zones 0)
     (modules 28)
@@
   (segment (start 190.853553 66.946447) (end 191 66.8) (width 0.2) (layer B.Cu) (net 20))
   (segment (start 191.2 67.77868) (end 191.136396 67.842284) (width 0.2) (layer B.Cu) (net 20))
+  (segment (start 194.575736 68.624264) (end 192.974874 70.225126) (width 0.15) (layer B.Cu) (net 21))
+  (segment (start 192.974874 70.225126) (end 192.974874 70.246447) (width 0.15) (layer B.Cu) (net 21))
   (segment (start 193.257716 69.963604) (end 193.257716 69.942284) (width 0.2) (layer B.Cu) (net 21))
+  (segment (start 193.975736 68.024264) (end 193.975736 68.538478) (width 0.15) (layer B.Cu) (net 22))
+  (segment (start 193.975736 68.538478) (end 192.798097 69.716117) (width 0.15) (layer B.Cu) (net 22))
+  (segment (start 194.4 69.3) (end 187.6 69.3) (width 0.15) (layer F.Cu) (net 23))
+  (segment (start 187.6 69.3) (end 186.85 68.55) (width 0.15) (layer F.Cu) (net 23))
+  (segment (start 194.5 69.4) (end 194.4 69.3) (width 0.15) (layer F.Cu) (net 23))
+  (segment (start 194.8 69.4) (end 194.5 69.4) (width 0.15) (layer F.Cu) (net 23))
+  (via (at 194.8 69.4) (size 0.6) (drill 0.4) (layers F.Cu B.Cu) (net 23))
+  (segment (start 194.8 69.694112) (end 194.8 69.4) (width 0.15) (layer B.Cu) (net 23))
+  (segment (start 193.257716 71.236396) (end 194.8 69.694112) (width 0.15) (layer B.Cu) (net 23))
   (segment (start 186.059989 67.759989) (end 186.550001 68.250001) (width 0.15) (layer B.Cu) (net 23))
   (segment (start 186.550001 68.250001) (end 186.85 68.55) (width 0.15) (layer B.Cu) (net 23))
@@
   (segment (start 173.8 62.6) (end 175.7 62.6) (width 0.15) (layer B.Cu) (net 23))
   (segment (start 176.334999 63.234999) (end 177.00734 63.234999) (width 0.15) (layer B.Cu) (net 23))
-  (segment (start 186.85 68.55) (end 189.45 68.55) (width 0.15) (layer F.Cu) (net 23))
   (via (at 186.85 68.55) (size 0.6) (drill 0.4) (layers F.Cu B.Cu) (net 23))
   (segment (start 189.85 65) (end 189.85 67.82868) (width 0.15) (layer B.Cu) (net 25))
@@
   (segment (start 184.15 65.5) (end 184.15 66.05) (width 0.15) (layer B.Cu) (net 32))
   (segment (start 189.262563 68.655456) (end 189.262563 68.584761) (width 0.2) (layer B.Cu) (net 34))
+  (segment (start 194.875736 70) (end 195.3 70) (width 0.15) (layer F.Cu) (net 35))
+  (segment (start 194.637798 70) (end 194.875736 70) (width 0.15) (layer F.Cu) (net 35))
+  (segment (start 187.05 69.6) (end 194.237798 69.6) (width 0.15) (layer F.Cu) (net 35))
+  (segment (start 186 68.55) (end 187.05 69.6) (width 0.15) (layer F.Cu) (net 35))
+  (segment (start 194.237798 69.6) (end 194.637798 70) (width 0.15) (layer F.Cu) (net 35))
+  (segment (start 195.424264 67.775736) (end 195.67175 68.023222) (width 0.15) (layer B.Cu) (net 35))
+  (segment (start 195.67175 68.023222) (end 195.67175 69.62825) (width 0.15) (layer B.Cu) (net 35))
+  (segment (start 195.67175 69.62825) (end 195.6 69.7) (width 0.15) (layer B.Cu) (net 35))
+  (segment (start 195.6 69.7) (end 195.3 70) (width 0.15) (layer B.Cu) (net 35))
+  (via (at 195.3 70) (size 0.6) (drill 0.4) (layers F.Cu B.Cu) (net 35))
   (segment (start 184.05 68.05) (end 185.5 68.05) (width 0.15) (layer B.Cu) (net 35))
   (segment (start 185.5 68.05) (end 186 68.55) (width 0.15) (layer B.Cu) (net 35))
@@
   (segment (start 174.35 66.35) (end 174.35 66.05) (width 0.15) (layer B.Cu) (net 35))
   (segment (start 176.872001 64.865001) (end 176.915001 64.822001) (width 0.15) (layer B.Cu) (net 35))
+  (segment (start 185.449999 68.899999) (end 185.15 68.6) (width 0.15) (layer F.Cu) (net 36))
+  (segment (start 194.127661 69.9) (end 186.45 69.9) (width 0.15) (layer F.Cu) (net 36))
+  (segment (start 194.742663 70.515002) (end 194.127661 69.9) (width 0.15) (layer F.Cu) (net 36))
+  (segment (start 195.684998 70.515002) (end 194.742663 70.515002) (width 0.15) (layer F.Cu) (net 36))
+  (segment (start 196.1 70.1) (end 195.684998 70.515002) (width 0.15) (layer F.Cu) (net 36))
+  (segment (start 186.45 69.9) (end 185.449999 68.899999) (width 0.15) (layer F.Cu) (net 36))
+  (segment (start 194.824264 67.175736) (end 195.177816 66.822184) (width 0.15) (layer B.Cu) (net 36))
+  (segment (start 195.177816 66.822184) (end 195.34047 66.822184) (width 0.15) (layer B.Cu) (net 36))
+  (segment (start 195.34047 66.822184) (end 196.1 67.581714) (width 0.15) (layer B.Cu) (net 36))
+  (segment (start 196.1 67.581714) (end 196.1 70.1) (width 0.15) (layer B.Cu) (net 36))
+  (via (at 196.1 70.1) (size 0.6) (drill 0.4) (layers F.Cu B.Cu) (net 36))
   (segment (start 182.75 67.2) (end 184.15 68.6) (width 0.15) (layer B.Cu) (net 36))
   (via (at 185.15 68.6) (size 0.6) (drill 0.4) (layers F.Cu B.Cu) (net 36))

Commit message: Reloaded netlist. Added notes to F.Fab layer. Generated production files.
Parts:
- C1, C4: value C -> 1u
- C3, C5: value C -> 0u1
Other:
- board text added: "COMPONENT POSITION ORIGIN"
- board text added: "NOTES: 1. FOOTPRINTS ORIENTED PER IPC-7351FC LEVEL B (PIN 1 IN LOWER LEFT) 2. COMPONENT ROTATION IN DEGREES COUNTER-CLOCKWISE 3. ALL COMPONENTS MOUNTED ON B.CU LAYER (LED IS BOTTOM-MOUNT) 4. PCB IS 1.6mm FR4 RATED FOR ROHS REFLOW, 1OZ COPPER, ENIG FINISH 5. MATTE BLACK SOLDER MASK WITH WHITE SILKSCREEN 6. SOLDER PASTE MUST BE ROHS COMPLIANT (LEAD-FREE) 7. NO MARKS (E-TEST, QA, SERIAL NUMBER, ETC)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"
- board text added: "ROUTE BOARD OUTLINE EXCEPT TWO ENDS"
- board text added: "V-SCORE PARALLEL ENDS"
Changed lines of the file:
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@@
   (general
     (links 73)
-    (no_connects 13)
-    (area 151.126667 58.081428 208.589752 82.489752)
+    (no_connects 8)
+    (area 139 41.8 235.857146 119.825)
     (thickness 1.6)
-    (drawings 45)
+    (drawings 71)
     (tracks 391)
     (zones 0)
@@
     (47 F.CrtYd user)
     (48 B.Fab user hide)
-    (49 F.Fab user hide)
+    (49 F.Fab user)
   )
   (setup
@@
     (pad_to_mask_clearance 0)
     (aux_axis_origin 0 0)
-    (grid_origin 195 70)
+    (grid_origin 153.25 79)
     (visible_elements FFFFEF7F)
     (pcbplotparams
-      (layerselection 0x00004_00000000)
+      (layerselection 0x210fc_80000001)
       (usegerberextensions false)
       (excludeedgelayer true)
@@
       (drillshape 0)
       (scaleselection 1)
-      (outputdirectory ""))
+      (outputdirectory ../../../NeuroTinker_RFQ_Sept2017/NeuroBytes_Tonic_Neuron/))
   )
   (net 0 "")
@@
     (at 161.2 64.6 270)
     (descr 2)
+    (attr smd)
     (fp_text reference Q3 (at 0 -2.8 270) (layer Cmts.User)
       (effects (font (size 1 1) (thickness 0.15)))
@@
   (module KiCad_Footprints:ZF_LOGO_Tonic_Neuron (layer F.Cu)
     (at 167.5 65.25)
+    (attr smd)
     (fp_text reference G*** (at 0 0) (layer F.SilkS) hide
       (effects (font (thickness 0.3)))
@@
   (module KiCad_Footprints:ZF_IC_UFQFPN28-050 (layer B.Cu)
     (at 190.5 70.6 315)
+    (attr smd)
     (fp_text reference U1 (at 0 0 315) (layer B.Fab)
       (effects (font (size 1 1) (thickness 0.15)) (justify mirror))
@@
     (at 193.2 76.3 270)
     (descr 2)
+    (attr smd)
     (fp_text reference U2 (at 0 -2.8 270) (layer B.Fab)
       (effects (font (size 1 1) (thickness 0.15)) (justify mirror))
@@
   (module KiCad_Footprints:ZF_CONN_1-2_pad (layer F.Cu)
     (at 160.4 75)
+    (attr smd)
     (fp_text reference TP4 (at 0 1.5) (layer Cmts.User)
       (effects (font (size 1 1) (thickness 0.15)))
     )
-    (fp_text value TEST (at 0 -1.6) (layer F.Fab)
+    (fp_text value TEST (at 0 -1.6) (layer F.Fab) hide
       (effects (font (size 1 1) (thickness 0.15)))
     )
@@
   (module KiCad_Footprints:ZF_SMD_NonPol_0603 (layer B.Cu)
     (at 195.75 76.3 270)
+    (attr smd)
     (fp_text reference C1 (at 0 -1.5 270) (layer B.Fab)
       (effects (font (size 1 1) (thickness 0.15)) (justify mirror))
     )
-    (fp_text value C (at 0 4.7 270) (layer B.Fab) hide
+    (fp_text value 1u (at 0 4.7 270) (layer B.Fab) hide
       (effects (font (size 1 1) (thickness 0.15)) (justify mirror))
     )
@@
   (module KiCad_Footprints:ZF_SMD_NonPol_0402_cap (layer B.Cu)
     (at 188.85 76.1 90)
+    (attr smd)
     (fp_text reference C3 (at 0 -1.25 90) (layer B.Fab)
       (effects (font (size 1 1) (thickness 0.15)) (justify mirror))
     )
-    (fp_text value C (at 0 1.5 90) (layer B.Fab) hide
+    (fp_text value 0u1 (at 0 1.5 90) (layer B.Fab) hide
       (effects (font (size 1 1) (thickness 0.15)) (justify mirror))
     )
@@
   (module KiCad_Footprints:ZF_SMD_NonPol_0603 (layer B.Cu)
     (at 190.6 76.3 270)
+    (attr smd)
     (fp_text reference C4 (at 0 -1.5 270) (layer B.Fab)
       (effects (font (size 1 1) (thickness 0.15)) (justify mirror))
     )
-    (fp_text value C (at 0 4.7 270) (layer B.Fab) hide
+    (fp_text value 1u (at 0 4.7 270) (layer B.Fab) hide
       (effects (font (size 1 1) (thickness 0.15)) (justify mirror))
     )
@@
   (module KiCad_Footprints:ZF_SMD_NonPol_0402_cap (layer B.Cu)
     (at 191.6 65.7 180)
+    (attr smd)
     (fp_text reference C5 (at 0 -1.25 180) (layer B.Fab)
       (effects (font (size 1 1) (thickness 0.15)) (justify mirror))
     )
-    (fp_text value C (at 0 1.5 180) (layer B.Fab) hide
+    (fp_text value 0u1 (at 0 1.5 180) (layer B.Fab) hide
       (effects (font (size 1 1) (thickness 0.15)) (justify mirror))
     )
@@
   (module KiCad_Footprints:ZF_SMD_NonPol_0402 (layer B.Cu)
     (at 171.5 65.9 90)
+    (attr smd)
     (fp_text reference R1 (at 0 -1.5 90) (layer B.Fab)
       (effects (font (size 1 1) (thickness 0.15)) (justify mirror))
@@
   (module KiCad_Footprints:ZF_SMD_NonPol_0402 (layer B.Cu)
     (at 186.2 74.3)
+    (attr smd)
     (fp_text reference R2 (at 0 -1.5) (layer B.Fab)
       (effects (font (size 1 1) (thickness 0.15)) (justify mirror))
@@
   (module KiCad_Footprints:ZF_SMD_NonPol_0402 (layer B.Cu)
     (at 186.2 72 180)
+    (attr smd)
     (fp_text reference R3 (at 0 -1.5 180) (layer B.Fab)
       (effects (font (size 1 1) (thickness 0.15)) (justify mirror))
@@
   (module KiCad_Footprints:ZF_SMD_NonPol_0402 (layer B.Cu)
     (at 191.6 66.8 180)
+    (attr smd)
     (fp_text reference R4 (at 0 -1.5 180) (layer B.Fab)
       (effects (font (size 1 1) (thickness 0.15)) (justify mirror))
@@
   (module KiCad_Footprints:ZF_SMD_NonPol_0402 (layer B.Cu)
     (at 171.5 63.5 270)
+    (attr smd)
     (fp_text reference R5 (at 0 -1.5 270) (layer B.Fab)
       (effects (font (size 1 1) (thickness 0.15)) (justify mirror))
@@
   (module KiCad_Footprints:ZF_SMD_NonPol_0402 (layer B.Cu)
     (at 163.5 64.6 270)
+    (attr smd)
     (fp_text reference R6 (at 0 -1.5 270) (layer B.Fab)
       (effects (font (size 1 1) (thickness 0.15)) (justify mirror))
@@
   (module KiCad_Footprints:ZF_CONN_1-2_pad (layer F.Cu)
     (at 177.6 71.6)
+    (attr smd)
     (fp_text reference TP3 (at 0 1.5) (layer Cmts.User)
       (effects (font (size 1 1) (thickness 0.15)))
     )
-    (fp_text value TEST (at 0 -1.6) (layer F.Fab)
+    (fp_text value TEST (at 0 -1.6) (layer F.Fab) hide
       (effects (font (size 1 1) (thickness 0.15)))
     )
@@
     (at 192.7 62.85)
     (attr smd)
-    (fp_text reference SW1 (at -0.1 -1.65) (layer F.Fab)
+    (fp_text reference SW1 (at -0.1 -1.65) (layer F.Fab) hide
       (effects (font (size 1 1) (thickness 0.15)))
     )
@@
     (at 173.4 65.2)
     (descr 2)
+    (attr smd)
     (fp_text reference Q1 (at 0 -2.8) (layer Cmts.User)
       (effects (font (size 1 1) (thickness 0.15)))
@@
     (at 176.4 65.2)
     (descr 2)
+    (attr smd)
     (fp_text reference Q2 (at 0 -2.8) (layer Cmts.User)
       (effects (font (size 1 1) (thickness 0.15)))
@@
   (module KiCad_Footprints:ZF_SMD_NonPol_0402 (layer B.Cu)
     (at 195 68.2 225)
+    (attr smd)
     (fp_text reference R7 (at 0 -1.5 225) (layer B.Fab)
       (effects (font (size 1 1) (thickness 0.15)) (justify mirror))
@@
   (module KiCad_Footprints:ZF_SMD_NonPol_0402 (layer B.Cu)
     (at 194.4 67.6 225)
+    (attr smd)
     (fp_text reference R8 (at 0 -1.5 225) (layer B.Fab)
       (effects (font (size 1 1) (thickness 0.15)) (justify mirror))
@@
   (module KiCad_Footprints:ZF_SMD_NonPol_0402 (layer B.Cu)
     (at 173.2 62.6)
+    (attr smd)
     (fp_text reference R9 (at 0 -1.5) (layer B.Fab)
       (effects (font (size 1 1) (thickness 0.15)) (justify mirror))
@@
   (module KiCad_Footprints:ZF_SMD_nonpol_1206 (layer B.Cu)
     (at 187 78 180)
+    (attr smd)
     (fp_text reference C2 (at 0 -1.75 180) (layer B.Fab)
       (effects (font (size 1 1) (thickness 0.15)) (justify mirror))
@@
       (net 2 GND))
   )
+  (gr_line (start 157.25 45) (end 162.25 45) (layer F.Fab) (width 0.2))
+  (gr_line (start 151.25 68) (end 151.25 66) (layer F.Fab) (width 0.2))
+  (gr_line (start 151.25 68) (end 149.25 68) (layer F.Fab) (width 0.2))
+  (gr_line (start 151.25 65) (end 151.25 65) (layer F.Fab) (width 0.2))
+  (gr_line (start 147.25 64) (end 151.25 68) (layer F.Fab) (width 0.2))
+  (gr_line (start 147.25 55) (end 147.25 64) (layer F.Fab) (width 0.2))
+  (gr_line (start 157.25 45) (end 147.25 55) (layer F.Fab) (width 0.2))
+  (gr_line (start 207.25 68) (end 209.25 68) (layer F.Fab) (width 0.2))
+  (gr_line (start 207.25 68) (end 207.25 66) (layer F.Fab) (width 0.2))
+  (gr_line (start 211.25 64) (end 207.25 68) (layer F.Fab) (width 0.2))
+  (gr_line (start 211.25 55) (end 211.25 64) (layer F.Fab) (width 0.2))
+  (gr_line (start 201.25 45) (end 211.25 55) (layer F.Fab) (width 0.2))
+  (gr_line (start 193.25 45) (end 201.25 45) (layer F.Fab) (width 0.2))
+  (gr_line (start 162.25 45) (end 193.25 45) (layer F.Fab) (width 0.2))
+  (gr_text "V-SCORE PARALLEL ENDS" (at 178.25 43) (layer F.Fab)
+    (effects (font (size 1.5 1.5) (thickness 0.3)))
+  )
+  (gr_line (start 189.25 80) (end 191.25 80) (layer F.Fab) (width 0.2))
+  (gr_line (start 189.25 80) (end 189.25 82) (layer F.Fab) (width 0.2))
+  (gr_line (start 196.25 87) (end 189.25 80) (layer F.Fab) (width 0.2))
+  (gr_line (start 224.25 87) (end 196.25 87) (layer F.Fab) (width 0.2))
+  (gr_text "ROUTE BOARD OUTLINE\nEXCEPT TWO ENDS" (at 210.25 84) (layer F.Fab)
+    (effects (font (size 1.5 1.5) (thickness 0.3)))
+  )
+  (gr_line (start 161.25 87) (end 181.25 87) (layer F.Fab) (width 0.2))
+  (gr_line (start 154.25 80) (end 161.25 87) (layer F.Fab) (width 0.2))
+  (gr_line (start 154.25 80) (end 156.25 80) (layer F.Fab) (width 0.2))
+  (gr_line (start 154.25 80) (end 154.25 82) (layer F.Fab) (width 0.2))
+  (gr_text "COMPONENT\nPOSITION ORIGIN" (at 171.25 84) (layer F.Fab)
+    (effects (font (size 1.5 1.5) (thickness 0.3)))
+  )
+  (gr_text "NOTES:\n1. FOOTPRINTS ORIENTED PER IPC-7351FC LEVEL B (PIN 1 IN LOWER LEFT)\n2. COMPONENT ROTATION IN DEGREES COUNTER-CLOCKWISE\n3. ALL COMPONENTS MOUNTED ON B.CU LAYER (LED IS BOTTOM-MOUNT)\n4. PCB IS 1.6mm FR4 RATED FOR ROHS REFLOW, 1OZ COPPER, ENIG FINISH\n5. MATTE BLACK SOLDER MASK WITH WHITE SILKSCREEN\n6. SOLDER PASTE MUST BE ROHS COMPLIANT (LEAD-FREE)\n7. NO MARKS (E-TEST, QA, SERIAL NUMBER, ETC) ON FRONT (LOGO SIDE) OF BOARD\n8. BOARDS TO BE SHIPPED IN CUSTOMER-SUPPLIED FOAM TRAYS\n9. 3MM LED HOLE IS PLATED" (at 139 107) (layer F.Fab)
+    (effects (font (size 1.5 1.5) (thickness 0.3)) (justify left))
+  )
   (gr_text POWER (at 182.9 67.5) (layer B.SilkS)
