File: HARDWARE/NeuroBytes_Tonic_Neuron.sch (KiCad schematic (older format))
At the start: 28 parts, among them P1 CONN_01X04, P2 CONN_01X04, P3 CONN_01X04, P4 JST_GH_5-pos, Q1 Q_NPN_BEC, Q2 Q_NPN_BEC, Q3 Q_NPN_BEC, SW1 SW_PUSH, U1 STM32L011Gx, U2 TLV70033_SOT23-5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

Commit message: generated fab files and BOM
Parts:
- U2: Link (none) -> https://www.digikey.com/product-detail/en/on-semiconductor/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; Mfr (none) -> ON Semiconductor; Mfr Part # (none) -> NCP114BSN330T1G; Package (none) -> SOT23-5L; Subs Allowed No -> Yes
- U3: Link (none) -> https://www.digikey.com/product-detail/en/semtech-corporati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; Mfr (none) -> Semtech Corporation; Mfr Part # (none) -> RCLAMP0503F.TCT; Package (none) -> 5-TSSOP
Changed lines of the file:
@@
 F 2 "KiCad_Footprints:ZF_SOT23-5L" H 13850 6075 50  0001 C CIN
 F 3 "" H 13850 5800 50  0001 C CNN
-F 4 "No" H 13850 5750 60  0001 C CNN "Subs Allowed"
-F 5 "Yes" H 13850 5750 60  0001 C CNN "RoHS"
+F 4 "ON Semiconductor" H 13850 5750 60  0001 C CNN "Mfr"
+F 5 "NCP114BSN330T1G" H 13850 5750 60  0001 C CNN "Mfr Part #"
+F 6 "SOT23-5L" H 13850 5750 60  0001 C CNN "Package"
+F 7 "https://www.digikey.com/product-detail/en/on-semiconductor/NCP114BSN330T1G/NCP114BSN330T1GOSTR-ND/6560606" H 13850 5750 60  0001 C CNN "Link"
+F 8 "Yes" H 13850 5750 60  0001 C CNN "Subs Allowed"
+F 9 "Yes" H 13850 5750 60  0001 C CNN "RoHS"
 	1    13850 5750
 	1    0    0    -1
@@
 F 2 "KiCad_Footprints:ZF_SMD_SOT-353" H 6900 2050 60  0001 C CNN
 F 3 "" H 6900 2050 60  0001 C CNN
-F 4 "No" H 6750 2200 60  0001 C CNN "Subs Allowed"
-F 5 "Yes" H 6750 2200 60  0001 C CNN "RoHS"
+F 4 "Semtech Corporation" H 6750 2200 60  0001 C CNN "Mfr"
+F 5 "RCLAMP0503F.TCT" H 6750 2200 60  0001 C CNN "Mfr Part #"
+F 6 "5-TSSOP" H 6750 2200 60  0001 C CNN "Package"
+F 7 "https://www.digikey.com/product-detail/en/semtech-corporation/RCLAMP0503F.TCT/RCLAMP0503F.TCTTR-ND/5113629" H 6750 2200 60  0001 C CNN "Link"
+F 8 "No" H 6750 2200 60  0001 C CNN "Subs Allowed"
+F 9 "Yes" H 6750 2200 60  0001 C CNN "RoHS"
 	1    6750 2200
 	-1   0    0    1

Commit message: updated footprints to include B.Fab outlines. minor routing changes. poured ground plane around connectors. re-generated Gerbers. added placement pdf.
Parts:
- C1, C4: footprint KiCad_Footprints:ZF_SMD_NonPol_0603 -> Capacitors_SMD:C_0603_HandSoldering
- C2: footprint KiCad_Footprints:ZF_SMD_nonpol_1206 -> Capacitors_SMD:C_1206
Changed lines of the file:
@@
 F 0 "C1" H 13025 6000 50  0000 L CNN
 F 1 "1u" H 13025 5800 50  0000 L CNN
-F 2 "KiCad_Footprints:ZF_SMD_NonPol_0603" H 13038 5750 50  0001 C CNN
+F 2 "Capacitors_SMD:C_0603_HandSoldering" H 13038 5750 50  0001 C CNN
 F 3 "" H 13000 5900 50  0000 C CNN
 F 4 "Taiyo Yuden" H 13000 5900 60  0001 C CNN "Mfr"
@@
 F 0 "C2" H 1925 5900 50  0000 L CNN
 F 1 "10u" H 1925 5700 50  0000 L CNN
-F 2 "KiCad_Footprints:ZF_SMD_nonpol_1206" H 1938 5650 50  0001 C CNN
+F 2 "Capacitors_SMD:C_1206" H 1938 5650 50  0001 C CNN
 F 3 "" H 1900 5800 50  0001 C CNN
 F 4 "Taiyo Yuden" H 1900 5800 60  0001 C CNN "Mfr"
@@
 F 0 "C4" H 14675 6000 50  0000 L CNN
 F 1 "1u" H 14675 5800 50  0000 L CNN
-F 2 "KiCad_Footprints:ZF_SMD_NonPol_0603" H 14688 5750 50  0001 C CNN
+F 2 "Capacitors_SMD:C_0603_HandSoldering" H 14688 5750 50  0001 C CNN
 F 3 "" H 14650 5900 50  0000 C CNN
 F 4 "Taiyo Yuden" H 14650 5900 60  0001 C CNN "Mfr"
